Commit message: adjusted lidar position

File: urdf/bot.urdf (robot description, URDF)
Before this commit: robot bot, 4 links, 3 joints
Links:
- removed link laser
- added link velodyne
Joints:
- joint j_laser: child laser -> velodyne; origin xyz=0 0 0 rpy=0 0 0 -> xyz=0 0 0 rpy=0 0.05 0

Commit message: deployment modification

File: urdf/bot.urdf (robot description, URDF)
Before this commit: robot bot, 4 links, 3 joints
Links:
- removed link imu_link
- added link imu_base
Joints:
- joint j_imu: child imu_link -> imu_base; origin xyz=0 0 0 rpy=0 0 0 -> xyz=0 0 0 rpy=0 0.05 0
- joint j_laser: origin xyz=0 0 0 rpy=0 0 0 -> xyz=0 0 0 rpy=0 0.05 0
